Commit message: Modify pointreg, not finished

File: src/turtle_bot_description/description/robot.urdf.xacro (robot description, xacro)
@@ -7,5 +7,5 @@
     <xacro:arg name="robot_material_color_rgb" default="0 1 0 1"/>
     <xacro:include filename="$(find turtle_bot_description)/description/xacro/inertial_macros.xacro" />
-    <!-- <xacro:include filename="$(find turtle_bot_description)/description/xacro/imu_sensor.xacro" /> -->
+    <xacro:include filename="$(find turtle_bot_description)/description/xacro/imu_sensor.xacro" />
     <!-- xacro:include filename="$(find turtle_bot_description)/description/xacro/depth_camera.xacro" / -->
     <xacro:include filename="$(find turtle_bot_description)/description/xacro/gazebo_control.xacro" />

File: src/turtle_bot_description/description/xacro/imu_sensor.xacro (robot description, xacro)
@@ -4,10 +4,10 @@
   <visual>
     <geometry>
-      <box size="0.1 0.1 0.1"/>
+      <box size="0.01 0.01 0.01"/>
     </geometry>
   </visual>
   <collision>
     <geometry>
-      <box size="0.1 0.1 0.1"/>
+      <box size="0.01 0.01 0.01"/>
     </geometry>
   </collision>
@@ -29,5 +29,5 @@
         </ros>
         <initial_orientation_as_reference>false</initial_orientation_as_reference>
-        <frame_name>imu_link</frame_name>
+        <frame_name>$(arg namespace)/imu_link</frame_name>
       </plugin>
       <always_on>true</always_on>
