Commit message: Add Registration base on PointLK

File: src/livox_sim/urdf/mid360.xacro (robot description, xacro)
@@ -3,5 +3,5 @@
   <xacro:property name="M_PI" value="3.1415926"/>
   <xacro:property name="laser_min_range" value="0.1"/>
-  <xacro:property name="laser_max_range" value="200.0"/>
+  <xacro:property name="laser_max_range" value="10.0"/>
   <xacro:property name="samples" value="40000"/>
   <xacro:property name="resolution" value="0.002"/>

Commit message: Push for remote development

File: src/livox_sim/urdf/mid360.xacro (robot description, xacro)
@@ -7,5 +7,5 @@
   <xacro:property name="resolution" value="0.002"/>
   <xacro:property name="noise_mean" value="0.0"/>
-  <xacro:property name="noise_stddev" value="0.01"/>
+  <xacro:property name="noise_stddev" value="0.0"/>
   <xacro:property name="mass" value="0.4" />
   <xacro:property name="length" value="0.1" />

Commit message: Add turtule bot model for better wheel odometry

File: src/livox_sim/urdf/mid360.xacro (robot description, xacro)
@@ -9,7 +9,7 @@
   <xacro:property name="noise_stddev" value="0.0"/>
   <xacro:property name="mass" value="0.4" />
-  <xacro:property name="length" value="0.1" />
-  <xacro:property name="width" value="0.06" />
-  <xacro:property name="height" value="0.06" />
+  <xacro:property name="length" value="0.03" />
+  <xacro:property name="width" value="0.03" />
+  <xacro:property name="height" value="0.03" />
   <xacro:macro name="box_inertia" params="m w h d">
     <inertial>

Commit message: Filter ground points, no effect, try pointlk

File: src/livox_sim/urdf/mid360.xacro (robot description, xacro)
@@ -3,5 +3,5 @@
   <xacro:property name="M_PI" value="3.1415926"/>
   <xacro:property name="laser_min_range" value="0.1"/>
-  <xacro:property name="laser_max_range" value="10.0"/>
+  <xacro:property name="laser_max_range" value="5.0"/>
   <xacro:property name="samples" value="40000"/>
   <xacro:property name="resolution" value="0.002"/>
