Commit message: Modify livox resolution and add transformation restriction for point_reg

File: src/livox_sim/urdf/mid360 copy.xacro (robot description, xacro)
@@ -4,6 +4,6 @@
   <xacro:property name="laser_min_range" value="0.1"/>
   <xacro:property name="laser_max_range" value="5.0"/>
-  <xacro:property name="samples" value="20000"/>
-  <xacro:property name="resolution" value="0.02"/>
+  <xacro:property name="samples" value="40000"/>
+  <xacro:property name="resolution" value="0.002"/>
   <xacro:property name="noise_mean" value="0.0"/>
   <xacro:property name="noise_stddev" value="0.0"/>
@@ -37,5 +37,5 @@
         <pose>0 0 0 0 0 0</pose>
         <visualize>true</visualize>
-        <update_rate>50</update_rate>
+        <update_rate>10</update_rate>
         <!-- This ray plgin is only for visualization. -->
         <plugin name="${name}_plugin" filename="libros2_livox.so">
@@ -49,8 +49,8 @@
 				</horizontal>
 				<vertical>
-          <samples>360</samples>
-          <resolution>1</resolution>
-          <min_angle>${-0.0/180*M_PI}</min_angle>
-          <max_angle>${55.22/180*M_PI}</max_angle>
+				<samples>360</samples>
+				<resolution>1</resolution>
+				<min_angle>${-7.22/180*M_PI}</min_angle>
+				<max_angle>${55.22/180*M_PI}</max_angle>
 				</vertical>
 			  </scan>
